File: boards/ToolTron_ToolBoxv2.0.brd (EAGLE design)
At the start: 88.9 x 54 mm, 37 parts, among them U1 ATTINY1634, U2 4N25SM, U3 MAX13082E, U4 MLX91206, U5 2N7000, U6 NCP1117DT50RKG, U7 NCP1117DT50RKG

Commit message: updated boards to include holes.
Routing:
- net GND: vias 2 -> 4
Changed lines of the file:
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@@
 <wire x1="22.5679" y1="21.5138" x2="26.5049" y2="21.5138" width="0.6096" layer="1"/>
 <wire x1="26.5049" y1="21.5138" x2="26.5049" y2="22.6568" width="0.6096" layer="1"/>
+<via x="84.1375" y="4.7625" extent="1-16" drill="3.2" diameter="6.4516"/>
+<via x="84.1375" y="49.2125" extent="1-16" drill="3.2" diameter="6.4516"/>
 </signal>
 <signal name="N$3">
